File: pica.kicad_pcb (KiCad board)
At the start: 2 copper layers, 114.3 x 96.5 mm, 118 parts, among them J1 CONN_02X03, J2 CONN_02X03, J3 CONN_02X03, J4 CONN_02X03, J5 CONN_02X03, M1 CONN_01X01, M2 CONN_01X01, M3 CONN_01X01, M4 CONN_01X01, P1 36-4966-ND, P10 CONN_02X06, P11 CONN_01X06, P12 CONN_01X02, P13 CONN_01X02, P14 CONN_01X02, P15 CONN_01X03, P19 CONN_01X04, P2 36-4966-ND, P20 CONN_01X04, P21 CONN_01X04, P22 CONN_01X04, P23 CONN_01X04, P24 CONN_01X04, P25 CONN_01X02, P26 CONN_01X02, P27 CONN_01X02, P28 CONN_01X02, P29 CONN_01X02, P3 36-4966-ND, P30 CONN_01X02, P32 CONN_02X03, P33 CONN_01X02, P34 CONN_01X02, P38 CONN_01X03, P4 36-4966-ND, P40 CONN_01X02, P5 CONN_02X03, P6 CONN_01X03, P7 CONN_01X04, P8 CONN_01X02, P9 CONN_02X04, Q1 IRFL024ZPbF, Q2 IRLML6346, Q3 IRFZ48VS, Q4 IRLML6346, Q5 IRFL024ZPbF, Q6 IRLML6346, SW1 BSF-3100, U1 LM2596-ADJ, U2 MC7805BDTRKG

Commit message: rev b
Parts:
- removed D1: D, Diodes_ThroughHole:Diode_DO-35_SOD27_Horizontal_RM10
- removed P12, P26, P34, P40: CONN_01X02, Pin_Headers:Pin_Header_Straight_1x02
- removed P32: CONN_02X03, Pin_Headers:Pin_Header_Straight_2x03
- removed P38: CONN_01X03, Pin_Headers:Pin_Header_Straight_1x03
- added D13: 1N5333, RAMPZ:Diode_Horizontal, F.Cu at (143.1, 105.3)
- added P16: CONN_02X02, Pin_Headers:Pin_Header_Straight_2x02, F.Cu at (155.8, 113.2)
- added P17: CONN_01X02, Pin_Headers:Pin_Header_Straight_1x02, F.Cu at (185.4, 110.5)
- added R12: 2K, Resistors_SMD:R_0805_HandSoldering, F.Cu at (157.9, 129.9)
- added R14: 4.7k, Resistors_SMD:R_0805_HandSoldering, F.Cu at (157.9, 135.0)
- added R15: 2K, Resistors_SMD:R_0805_HandSoldering, F.Cu at (142.5, 128.3)
- added R16: 4.7k, Resistors_SMD:R_0805_HandSoldering, F.Cu at (142.5, 130.8)
- C11: moved to B.Cu
- C13: value C_Small -> 15nF; footprint Capacitors_SMD:C_1206_HandSoldering -> Capacitors_SMD:C_0805_HandSoldering; moved to F.Cu
- C14: value 100UF -> 470u; footprint Capacitors_SMD:c_elec_6.3x5.8 -> Capacitors_ThroughHole:C_Radial_D10_L13_P5
- D2: value Led_Small -> GREEN
- D8: value SS36 -> MBRA340T3G
- L1: value 33uH -> 82uH
- P15: value CONN_01X03 -> CONN_02X02; footprint Pin_Headers:Pin_Header_Straight_1x03 -> Pin_Headers:Pin_Header_Straight_2x02
- P5: value CONN_02X03 -> CONN_02X06; footprint Pin_Headers:Pin_Header_Straight_2x03 -> Pin_Headers:Pin_Header_Straight_2x06
- P6: value CONN_01X03 -> JST-XH; footprint Pin_Headers:Pin_Header_Straight_1x03 -> RAMPZ:JST_XH_2POS
- P8: value CONN_01X02 -> JST-PH; footprint Pin_Headers:Pin_Header_Straight_1x02 -> RAMPZ:JST_PH_2POS
- Q2, Q4, Q6: value IRLML6346 -> IRLM6346; footprint TO_SOT_Packages_SMD:SOT-23 -> TO_SOT_Packages_SMD:SOT-23_Handsoldering
- R25: value 40.2K -> 17.2K
- R26: value 4.7K -> 2K
- R4: value 4.7k -> 2K
- RP1, RP2, RP3: footprint Resistors_SMD:R_Array_Convex_4x1206 -> RAMPZ:RESARY_4_CTS_744
- moved REF** 85.3 mm to (190.9, 80.6), turned to 0 degrees
- moved P8 46.5 mm to (121.1, 128.7), turned to 0 degrees
- moved P15 39.2 mm to (167.3, 113.3), turned to 180 degrees
- moved R26 26.8 mm to (209.0, 119.8), turned to 0 degrees
- moved C10 26.6 mm to (189.2, 102.1), turned to 0 degrees
- moved P6 23.3 mm to (121.4, 134.2)
- moved C13 21.1 mm to (203.6, 120.9), turned to 0 degrees
- moved R25 18.6 mm to (203.6, 118.6), turned to 0 degrees
- moved P5 17.6 mm to (107.7, 122.8), turned to 0 degrees
- moved RP2 15.8 mm to (179.1, 129.6), turned to 270 degrees
- moved C15 15.1 mm to (129.3, 102.0)
- moved C11 13.2 mm to (142.0, 99.0), turned to 270 degrees
- moved R11 12.7 mm to (179.1, 109.9), turned to 0 degrees
- moved D9 11.6 mm to (147.0, 94.1)
- moved R4 9.37 mm to (188.1, 76.3), turned to 0 degrees
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Connections:
- net /RX0 renamed RX0
- net Net-(D11-Pad2) renamed /Q3_D
- C11 pad 1: +VPSU -> /AM_VIN
- C12 pad 1: Net-(C12-Pad1) -> +VPSU
- C15 pad 1: Net-(C15-Pad1) -> VCC
- P15 pad 1: +5P -> +12V
- P15 pad 2: VCC -> /FE1_D
- P15 pad 3: Net-(C15-Pad1) -> +12V
- P5 pad 2: +12V -> +VPSU
- P5 pad 4: +12V -> +VPSU
- P6 pad 1: +3V3 -> GND
- P6 pad 2: Net-(P6-Pad2) -> +12V
- P8 pad 1: +12V -> GND
- P8 pad 2: /FE1_D -> +12V
- Q2 pad 2: /FE1_D -> GND
- Q2 pad 3: GND -> /FE1_D
- Q4 pad 2: Net-(Q4-Pad2) -> GND
- Q4 pad 3: GND -> Net-(Q4-Pad3)
- Q6 pad 2: /FE2_D -> GND
- Q6 pad 3: GND -> /FE2_D
- R4 pad 1: +12V -> /AM_VIN
- RL1 pad 4: Net-(Q4-Pad2) -> Net-(Q4-Pad3)
- RP2 pad 1: /FE2_G -> HOTEND_EN
- RP2 pad 2: /FE1_G -> FET3_EN
- RP2 pad 3: /HE2_G -> FAN_EN
- RP2 pad 4: /HE1_G -> FET5_EN
- RP3 pad 3: VAA -> +VPSU
- RP3 pad 4: VAA -> +VPSU
- SER0 pad 1: Net-(P6-Pad2) -> VCC
- SER0 pad 4: /TX0 -> Net-(R12-Pad1)
- SER1 pad 1: Net-(P6-Pad2) -> VCC
- SER1 pad 4: TX1 -> Net-(R15-Pad1)
- SHIELD1 pad 1: /TX0 -> TX0
- SHIELD1 pad 5V: +5P -> Net-(SHIELD1-Pad5V)
- U1 pad 1: Net-(C12-Pad1) -> +VPSU
- U2 pad 1: +VPSU -> /AM_VIN
- U2 pad 3: Net-(C15-Pad1) -> VCC
Routing:
- net +3V3: track 111.5 -> 0.00 mm, vias 1 -> 0
- net +12V: track 214.1 -> 113.0 mm, vias 4 -> 2
- net VCC: track 215.4 -> 124.4 mm
- net +5P: track 64.8 -> 0.00 mm
- net +VPSU: track 201.7 -> 142.0 mm, vias 1 -> 2
- net /AM_VIN: track 23.1 -> 69.2 mm
- net Net-(P6-Pad2): track 21.2 -> 0.00 mm
- net GND: track 132.6 -> 113.0 mm, vias 20 -> 24
- net Net-(C15-Pad1): track 17.4 -> 0.00 mm
- net Net-(D9-Pad2): track 7.05 -> 24.1 mm
- net /HE2_G: track 51.2 -> 34.2 mm
- net /Q3_D: track 75.3 -> 58.6 mm, vias 1 -> 4
- net TX1: track 17.5 -> 5.21 mm
- net Net-(C12-Pad1): track 12.3 -> 0.00 mm
- net FET5_EN: track 4.49 -> 16.4 mm
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- added copper zone on F.Cu, net +12V
- added copper zone on F.Cu, net /HE1_D
- added copper zone on F.Cu, net /HE2_D
- added copper zone on B.Cu, net /Q3_D
Other:
- board size 114.3 x 96.5 mm -> 114.3 x 94.9 mm
- board text added: "+SUP"
- board text added: "-SUP"
- board text added: "CC"
- board text added: "CONFIG"
- board text added: "Creative Commons Atribution-ShareAlike"
- board text added: "Design by mjrice"
- board text added: "E0"
- board text added: "E1"
- board text added: "PICA-PCB-REVB"
- board text added: "Power, Interface, and Control Adapter A Reprap Arduino Mega Pololu Shield"
- board text added: "VIN GND GND 5V 3.3V RST"
- board text added: "X"
- board text added: "Y"
- board text added: "Z"
- board text removed: "1"
- board text removed: "1-2 ARDU"
- board text removed: "2"
- board text removed: "2-3 U2"
- board text removed: "3"
- board text removed: "3.3V"
- board text removed: "E0-MOTOR"
- board text removed: "E1-MOTOR"
- board text removed: "INPUT 12-24V"
- board text removed: "INPUT SELECT"
- board text removed: "PICA REV A"
- board text removed: "SELECT"
- board text removed: "VCC SELECT JUMPER"
- board text removed: "X-MOTOR"
- board text removed: "Y-MOTOR"
- board text removed: "Z-MOTOR"

Commit message: Final rev C design files
Parts:
- added C16: .1UF, Capacitors_SMD:C_0805_HandSoldering, B.Cu at (150.1, 140.2)
- added P12: JST-PH, RAMPZ:JST_PH_2POS, F.Cu at (163.6, 112.1)
- added P18: JST-PH, RAMPZ:JST_PH_2POS, F.Cu at (152.5, 112.1)
- added P26: CONN_02X04, RAMPZ:PINHEADER_2X4_SMD, B.Cu at (143.3, 128.4)
- added R5: 4.7K, Resistors_SMD:R_0805_HandSoldering, F.Cu at (141.2, 135.0)
- added R6: 4.7K, Resistors_SMD:R_0805_HandSoldering, F.Cu at (128.0, 129.1)
- added U3: TLV70033DDC, SOT-23-5, B.Cu at (143.0, 128.8)
- C11, C6, C7, C8, C9: moved to F.Cu
- C12: value .1 -> .1UF; footprint Capacitors_SMD:C_1206_HandSoldering -> Capacitors_SMD:C_0805_HandSoldering
- P15, P16: value CONN_02X02 -> DUPONT; footprint Pin_Headers:Pin_Header_Straight_2x02 -> Pin_Headers:Pin_Header_Straight_1x02
- Q2, Q4, Q6: value IRLM6346 -> IRLML6346
- R1, R2, R3, R7: value 4.7k -> 4.7K; footprint Resistors_SMD:R_0805 -> Resistors_SMD:R_0805_HandSoldering
- R10: value 4.7K -> 2K
- R13, R14, R16: value 4.7k -> 4.7K
- R20, R21, R22, R23, R24: value 10K -> 4.7K
- R4: value 2K -> 4.7K; footprint Resistors_SMD:R_0805 -> Resistors_SMD:R_0805_HandSoldering
- RP1: value YC164-JR-0722RL -> YC164-JR-0733RL
- RP2: value YC164-JR-07100KL -> YC164-JR-07150KL; moved to F.Cu
- moved C6 7.43 mm to (130.9, 89.7), turned to 270 degrees
- moved R10 7.37 mm to (183.7, 129.1)
- moved P15 5.79 mm to (164.4, 108.3), turned to 90 degrees
- moved P16 5.54 mm to (153.3, 108.3), turned to 90 degrees
- moved C9 3.57 mm to (140.8, 79.3), turned to 180 degrees
- moved C11 3.39 mm to (145.4, 99.1)
- moved R2 2.62 mm to (133.7, 82.9)
- moved R7 2.24 mm to (131.5, 82.9)
- moved R8 1.86 mm to (180.0, 132.8)
- moved RP2 1.45 mm to (177.7, 129.1)
- moved C8 1.38 mm to (140.1, 83.0)
- moved R3 0.84 mm to (142.2, 82.9)
- moved R1 0.79 mm to (137.9, 82.9)
- moved Q4 0.73 mm to (180.2, 135.7), turned to 270 degrees
- moved REF** 0.61 mm to (191.4, 81.0)
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Connections:
- net Net-(R15-Pad1) renamed /TX1_S
- P15 pad 1: +12V -> /FE1_D
- P15 pad 2: /FE1_D -> +12V
- P16 pad 1: +12V -> /FE2_D
- P16 pad 2: /FE2_D -> +12V
- R11 pad 1: Net-(Q3-Pad1) -> BED_EN
- RP1 pad 1: FET5_EN -> FAN2_EN
- RP1 pad 3: FET3_EN -> HOTEND2_EN
- RP2 pad 2: FET3_EN -> FAN_EN
- RP2 pad 3: FAN_EN -> FAN2_EN
- RP2 pad 4: FET5_EN -> HOTEND2_EN
- SHIELD1 pad 10: FET3_EN -> HOTEND_EN
- SHIELD1 pad 11: FAN_EN -> Net-(SHIELD1-Pad11)
- SHIELD1 pad 12: FET5_EN -> Net-(SHIELD1-Pad12)
- SHIELD1 pad 2: Net-(SHIELD1-Pad2) -> HOTEND2_EN
- SHIELD1 pad 7: Net-(SHIELD1-Pad7) -> FAN2_EN
- SHIELD1 pad 9: HOTEND_EN -> FAN_EN
Routing:
- net Net-(C16-Pad1): track 0.00 -> 36.1 mm
- net HOTEND2_EN: track 0.00 -> 27.3 mm, vias 0 -> 1
- net /Q3_D: track 58.6 -> 80.2 mm
- net +12V: track 113.0 -> 91.8 mm
- net FAN2_EN: track 0.00 -> 21.2 mm
- net /TX1_S: track 9.62 -> 28.3 mm
- net BED_EN: track 17.6 -> 35.2 mm
- net FET5_EN: track 16.4 -> 0.00 mm
- net +VPSU: track 142.0 -> 127.6 mm
- net FET3_EN: track 12.8 -> 0.00 mm
- net GND: track 113.0 -> 104.5 mm, vias 24 -> 25
- net HOTEND_EN: track 12.2 -> 18.8 mm
- net SDA: track 10.7 -> 17.1 mm
- net THERM3: track 13.7 -> 18.9 mm
- net RX1: track 21.3 -> 26.4 mm
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Other:
- board text added: "(D7)"
- board text added: "(D9)"
- board text added: "FET2 (D10)"
- board text added: "FET3 (D2)"
- board text added: "FET4"
- board text added: "FET5"
- board text added: "MODEL"
- board text added: "PICA-PCB-REVC"
- board text added: "PWR ON"
- board text added: "RECOMMENDED CONNECTIONS HEATBED - FET1 HOTEND - FET2 PRINT FAN - FET4"
- board text removed: "CONFIG"
- board text removed: "DO NOT TOUCH"
- board text removed: "FET2 (D9)"
- board text removed: "FET3 (D10)"
- board text removed: "FET4 (D11)"
- board text removed: "FET5 (D12)"
- board text removed: "PICA-PCB-REVB"

Commit message: update rev e files
Parts:
- removed D7: SS36, Diodes_SMD:SMA_Handsoldering
- removed P15: DUPONT, Pin_Headers:Pin_Header_Straight_1x02
- removed REF**: Symbol_OSHW-Logo_SilkScreen, Symbols:Symbol_OSHW-Logo_SilkScreen
- removed RL1: SSR_2, RAMPZ:I4-PAC
- removed RP1: YC164-JR-0733RL, RAMPZ:RESARY_4_CTS_744
- removed RP3: YC164-JR-073K3L, RAMPZ:RESARY_4_CTS_744
- added C17: 10nF, Capacitors_SMD:C_1206_HandSoldering, F.Cu at (205.6, 137.7)
- added D1: SBRT20M60SP5-7, RAMPZ:POWERDI5, F.Cu at (192.5, 90.6)
- added F1: 0ZCJ0020FF2E, Fuse_Holders_and_Fuses:Fuse_SMD1206_Wave, F.Cu at (143.5, 89.2)
- added F2: 0ZCJ0020FF2E, Fuse_Holders_and_Fuses:Fuse_SMD1206_Wave, F.Cu at (107.0, 72.2)
- added F3: 0ZCJ0020FF2E, Fuse_Holders_and_Fuses:Fuse_SMD1206_Wave, F.Cu at (130.1, 139.8)
- added R17: 360, Resistors_SMD:R_0805_HandSoldering, F.Cu at (200.4, 127.9)
- added R18: 360, Resistors_SMD:R_0805_HandSoldering, F.Cu at (193.3, 138.9)
- added R19: 50, Resistors_SMD:R_0805_HandSoldering, F.Cu at (205.6, 131.7)
- added R27: 4.7K, Resistors_SMD:R_0805_HandSoldering, F.Cu at (150.0, 108.6)
- added R28: 4.7K, Resistors_SMD:R_0805_HandSoldering, F.Cu at (161.4, 108.7)
- added R29: 4.7K, Resistors_SMD:R_0805_HandSoldering, F.Cu at (147.4, 99.5)
- added R30: 4.7K, Resistors_SMD:R_0805_HandSoldering, F.Cu at (160.2, 100.3)
- added R31: 50, Resistors_SMD:R_0805_HandSoldering, F.Cu at (153.4, 102.3)
- added R32: 50, Resistors_SMD:R_0805_HandSoldering, F.Cu at (164.6, 102.3)
- added U4: MOC3061M, RAMPZ:6SMD, F.Cu at (188.3, 126.9)
- added U5: TRIAC, TO_SOT_Packages_SMD:TO-252-2Lead, F.Cu at (200.2, 131.4)
- C13: value 15nF -> 10nF; footprint Capacitors_SMD:C_0805_HandSoldering -> Capacitors_SMD:C_1206_HandSoldering
- D11: value SS36 -> MBR0560; footprint Diodes_SMD:SMA_Handsoldering -> Diodes_SMD:SOD-123
- EXP1, EXP2: footprint Connect:IDC_Header_Straight_10pins -> RAMPZ:IDC_Header_Straight_10pins_DUAL
- P12: value JST-PH -> JST-XH; footprint RAMPZ:JST_PH_2POS -> RAMPZ:JST_XH_2POS
- R10: value 2K -> 200
- R9: value 10 -> 50
- moved R8 6.55 mm to (177.3, 138.7), turned to 180 degrees
- moved P14 6.11 mm to (212.0, 125.3)
- moved P13 5.63 mm to (212.0, 131.1)
- moved D3 4.32 mm to (182.0, 136.3), turned to 90 degrees
- moved Q4 2.82 mm to (177.4, 135.3)
- moved CS1 2.19 mm to (205.6, 97.4)
- moved CS2 2.06 mm to (205.6, 81.3)
- moved P12 2.04 mm to (165.5, 112.7), turned to 90 degrees
- moved C9 2.00 mm to (138.8, 79.0)
- moved P3 1.93 mm to (212.2, 89.2)
- moved P4 1.91 mm to (212.2, 95.2)
- moved C6 1.91 mm to (129.0, 89.7)
- moved C7 1.91 mm to (133.9, 83.0)
- moved C8 1.91 mm to (138.2, 83.0)
- moved P9 1.91 mm to (139.4, 87.1)
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Connections:
- DRV_E0 pad 2: VCC -> /DRV_VCC
- DRV_E1 pad 2: VCC -> /DRV_VCC
- DRV_X1 pad 2: VCC -> /DRV_VCC
- DRV_Y1 pad 2: VCC -> /DRV_VCC
- DRV_Z1 pad 2: VCC -> /DRV_VCC
- J1 pad 1: VCC -> /DRV_VCC
- J1 pad 3: VCC -> /DRV_VCC
- J1 pad 5: VCC -> /DRV_VCC
- J2 pad 1: VCC -> /DRV_VCC
- J2 pad 3: VCC -> /DRV_VCC
- J2 pad 5: VCC -> /DRV_VCC
- J3 pad 1: VCC -> /DRV_VCC
- J3 pad 3: VCC -> /DRV_VCC
- J3 pad 5: VCC -> /DRV_VCC
- J4 pad 1: VCC -> /DRV_VCC
- J4 pad 3: VCC -> /DRV_VCC
- J4 pad 5: VCC -> /DRV_VCC
- J5 pad 1: VCC -> /DRV_VCC
- J5 pad 3: VCC -> /DRV_VCC
- J5 pad 5: VCC -> /DRV_VCC
- P5 pad 6: +12V -> Net-(F3-Pad1)
- P5 pad 8: +12V -> Net-(F3-Pad1)
- P6 pad 2: +12V -> Net-(F3-Pad1)
- P8 pad 2: +12V -> Net-(F3-Pad1)
- Q2 pad 1: /FE1_G -> FAN_EN
- Q6 pad 1: /FE2_G -> FAN2_EN
- R1 pad 1: VCC -> +5VL
- R2 pad 1: VCC -> +5VL
- R20 pad 1: VCC -> /DRV_VCC
- R21 pad 1: VCC -> /DRV_VCC
- R22 pad 1: VCC -> /DRV_VCC
- R23 pad 1: VCC -> /DRV_VCC
- R24 pad 1: VCC -> /DRV_VCC
- R3 pad 1: VCC -> +5VL
- R4 pad 1: /AM_VIN -> Net-(F1-Pad2)
- R7 pad 1: VCC -> +5VL
- SHIELD1 pad 5V: Net-(SHIELD1-Pad5V) -> +5VL
- SHIELD1 pad V_IN: /AM_VIN -> Net-(F1-Pad2)
Routing:
- net /DRV_VCC: track 0.00 -> 93.1 mm
- net VCC: track 127.8 -> 55.4 mm, vias 1 -> 0
- net /AM_VIN: track 68.9 -> 13.1 mm
- net Net-(F1-Pad2): track 0.00 -> 55.0 mm, vias 0 -> 1
- net /FE2_G: track 37.5 -> 0.00 mm, vias 1 -> 0
- net GND: track 104.5 -> 137.2 mm, vias 25 -> 24
- net /HE2_G: track 35.4 -> 3.82 mm, vias 1 -> 0
- net Net-(F3-Pad1): track 0.00 -> 30.3 mm
- net /FE1_G: track 23.4 -> 0.00 mm, vias 1 -> 0
- net FAN2_EN: track 21.2 -> 44.2 mm
- net Net-(D9-Pad2): track 24.1 -> 2.77 mm, vias 1 -> 0
- net HOTEND2_EN: track 27.3 -> 47.7 mm
- net /HE1_G: track 23.1 -> 3.01 mm, vias 1 -> 0
- net +VPSU: track 127.6 -> 147.7 mm, vias 2 -> 3
- net FAN_EN: track 10.7 -> 26.6 mm
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- added copper zone on F.Cu, net +5VL
- added copper zone on F.Cu, net /DRV_VCC
Other:
- board text added: "8 9 10 11 12 13 GND AREF"
- board text added: "ACIN"
- board text added: "ACLOAD"
- board text added: "AD15 AD14 AD13 AD12 AD11 AD10 AD9 AD8"
- board text added: "AD7 AD6 AD5 AD4 AD3 AD2 AD1 AD0"
- board text added: "ARDUINO PINS"
- board text added: "OSHW"
- board text added: "PA0"
- board text added: "PA6 PA4 PA2"
- board text added: "PA7 PA5 PA3 PA1"
- board text added: "PB0 PB2"
- board text added: "PB1 PB3"
- board text added: "PC0 PC2 PC4 PC6"
- board text added: "PC1 PC3 PC5 PC7"
- board text added: "PG0 PG2"
- board text added: "PG1 PD7"
- board text added: "PICA-PCB-REVE"
- board text added: "PL0 PL2 PL4 PL6"
- board text added: "PL1 PL3 PL5 PL7"
- board text added: "POWER INPUTS"
- board text added: "Power, Interface, and Control Adapter A Reprap Arduino Mega Pololu Shield https://github.com/mjrice/PICA"
- board text added: "RX0 TX0 2 3 4 5 6 7"
- board text added: "SCL SDA RX1 TX1 RX2 TX2 RX3 TX3"
- board text removed: "+SUP"
- board text removed: "-SUP"
- board text removed: "A"
- board text removed: "B"
- board text removed: "CAUTION!"
- board text removed: "HIGH VOLTAGE"
- board text removed: "PICA-PCB-REVC"
- board text removed: "Power, Interface, and Control Adapter A Reprap Arduino Mega Pololu Shield"
- board text removed: "SSR ON"
