File: pica.sch (KiCad schematic (older format))
At the start: 119 parts, among them J1 CONN_02X03, J2 CONN_02X03, J3 CONN_02X03, J4 CONN_02X03, J5 CONN_02X03, M1 CONN_01X01, M2 CONN_01X01, M3 CONN_01X01, M4 CONN_01X01, P1 36-4966-ND, P10 CONN_02X06, P11 CONN_01X06, P12 CONN_01X02, P13 CONN_01X02, P14 CONN_01X02, P15 CONN_01X03, P19 CONN_01X04, P2 36-4966-ND, P20 CONN_01X04, P21 CONN_01X04, P22 CONN_01X04, P23 CONN_01X04, P24 CONN_01X04, P25 CONN_01X02, P26 CONN_01X02, P27 CONN_01X02, P28 CONN_01X02, P29 CONN_01X02, P3 36-4966-ND, P30 CONN_01X02, P32 CONN_02X03, P33 CONN_01X02, P34 CONN_01X02, P38 CONN_01X03, P4 36-4966-ND, P40 CONN_01X02, P5 CONN_02X03, P6 CONN_01X03, P7 CONN_01X04, P8 CONN_01X02, P9 CONN_02X04, Q1 IRFL024ZPbF, Q2 IRLML6346, Q3 IRFZ48VS, Q4 IRLML6346, Q5 IRFL024ZPbF, Q6 IRLML6346, SW1 BSF-3100, U1 LM2596-ADJ, U2 MC7805BDTRKG

Commit message: added pdf of schematic
Other:
- note added: "Mounting holes"
- note removed: "Original pin assignments\nRS 16\nEN 17\nD4 23\nD5 25\nD6 27\nD7 29\nLCD_BEEPER 37\nBTN_EN1 31\nBTN_EN2 33\nBTN_ENC 35\nSDCARDDETECT 49"
- moved on the sheet: C6, C7, C8, C9, D3, M1, M2, M3, M4, P13, P14, Q4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

Commit message: rev b
Parts:
- removed D1: D, Diodes_ThroughHole:Diode_DO-35_SOD27_Horizontal_RM10, symbol D
- removed P12, P26, P34, P40: CONN_01X02, Pin_Headers:Pin_Header_Straight_1x02, symbol CONN_01X02
- removed P15, P38, P6: CONN_01X03, Pin_Headers:Pin_Header_Straight_1x03, symbol CONN_01X03
- removed P32, P5: CONN_02X03, Pin_Headers:Pin_Header_Straight_2x03, symbol CONN_02X03
- removed Q2, Q4, Q6: IRLML6346, TO_SOT_Packages_SMD:SOT-23, symbol Q_NMOS_GDS
- added D13: 1N5333, RAMPZ:Diode_Horizontal, symbol ZENER
- added P15, P16: CONN_02X02, Pin_Headers:Pin_Header_Straight_2x02, symbol CONN_02X02
- added P17: CONN_01X02, Pin_Headers:Pin_Header_Straight_1x02, symbol CONN_01X02
- added P5: CONN_02X06, Pin_Headers:Pin_Header_Straight_2x06, symbol CONN_02X06
- added P6: JST-XH, RAMPZ:JST_XH_2POS, symbol CONN_01X02
- added Q2, Q4, Q6: IRLM6346, TO_SOT_Packages_SMD:SOT-23_Handsoldering, symbol Q_NMOS_GSD
- added R12, R15: 2K, Resistors_SMD:R_0805_HandSoldering, symbol R
- added R14, R16: 4.7k, Resistors_SMD:R_0805_HandSoldering, symbol R
- C13: value C_Small -> 15nF; footprint Capacitors_SMD:C_1206_HandSoldering -> Capacitors_SMD:C_0805_HandSoldering
- C14: value 100UF -> 470u; footprint Capacitors_SMD:c_elec_6.3x5.8 -> Capacitors_ThroughHole:C_Radial_D10_L13_P5
- D2: value Led_Small -> GREEN
- D8: value SS36 -> MBRA340T3G
- L1: value 33uH -> 82uH
- P8: value CONN_01X02 -> JST-PH; footprint Pin_Headers:Pin_Header_Straight_1x02 -> RAMPZ:JST_PH_2POS
- R20, R21, R22, R23, R24: value 10K -> 4.7K
- R25: value 40.2K -> 17.2K
- R26: value 4.7K -> 2K
- R4: value 4.7k -> 4.7K
- RP1, RP2, RP3: footprint Resistors_SMD:R_Array_Convex_4x1206 -> RAMPZ:RESARY_4_CTS_744
Connections:
- net VAA is gone; now on net +VPSU: RP3.3 (P3), RP3.4 (P4)
- net +12V: now also P8.2 (P2), D13.1 (K), P15.1 (P1), P15.3 (P3), P16.1 (P1), P16.3 (P3), P17.1 (P1), P5.6 (P6), P5.8 (P8), P6.2 (P2); no longer P8.1 (P1), R4.1
- net +VPSU: now also C12.1, U1.1 (VIN), P17.2 (P2), P5.2 (P2), P5.4 (P4); no longer C11.1, U2.1 (VI)
- net AM_VIN: now also C11.1, R4.1, U2.1 (VI), D13.2 (A)
- net FAN_EN: now also RP2.3 (P3)
- net FE1_D: now also P15.2 (P2), P15.4 (P4), Q2.3 (D); no longer P8.2 (P2)
- net FE1_G: now also Q2.1 (G); no longer RP2.2 (P2)
- net FE2_D: now also P16.2 (P2), P16.4 (P4), Q6.3 (D)
- net FE2_G: now also Q6.1 (G); no longer RP2.1 (P1)
- net FET3_EN: now also RP2.2 (P2)
- net FET5_EN: now also RP2.4 (P4)
- net GND: now also P8.1 (P1), P5.1 (P1), P5.11 (P11), P5.3 (P3), P5.5 (P5), P5.7 (P7), P5.9 (P9), P6.1 (P1), Q2.2 (S), Q4.2 (S), Q6.2 (S), R14.2, R16.2
- net HE1_G: no longer RP2.4 (P4)
- net HE2_G: no longer RP2.3 (P3)
- net HOTEND_EN: now also RP2.1 (P1)
- net SSR_EN: now also Q4.1 (G)
- net TX0: now also R12.2; no longer SER0.4 (P4)
- net TX1: now also R15.2; no longer SER1.4 (P4)
- net VCC: now also C15.1, SER0.1 (P1), SER1.1 (P1), U2.3 (VO), P5.10 (P10), P5.12 (P12)
- net Q3_D: now reaches D11.2 (A), D4.1 (K), P28.1 (P1), P28.2 (P2), Q3.2 (D), Q3.4 (D)
- net at RL1.4: now also Q4.3 (D)
- net +5P: no longer names the net of SHIELD1.5V
- new net: R15.1, R16.1, SER1.4 (P4)
- new net: R12.1, R14.1, SER0.4 (P4)
Other:
- note added: "(TO HBP)"
- note added: "(TO HOTEND HEATER)"
- note added: "(TO PRINT FAN)"
- note added: "12V to 24V"
- note added: "24V to 12V switching regulator"
- note added: "455-1704-ND"
- note added: "455-2247-ND"
- note added: "5V Power for Shield"
- note added: "Combined output power from Q2, Q6, and U2 not to exceed 3A"
- note added: "Input Power Select\nInstall wire jumper if 12V input\n(do not install U1)\nOtherwise leave open"
- note added: "Install these parts only if power supply > 12V"
- note added: "Medium current MOSFET outputs (24V/5A)"
- note added: "Optional level translation on TX (out)"
- note added: "POWER INDUCTOR SRR1280-680M or MSS1278-683MLB"
- note added: "R25 = R26(VOUT/1.23-1)"
- note added: "Remove R14, R16 if interfacing to 5V serial device"
- note added: "Reset Button"
- note added: "Serial Expansion Ports"
- note added: "Thermistor / ADC Inputs"
- note added: "status leds"
- note removed: "12-24V"
- note removed: "12V 2-3"
- note removed: "1N4001"
- note removed: "22"
- note removed: ">12V 1-2"
- note removed: "Choose Regulator output\nor Arduino regulator output"
- note removed: "Green"
- note removed: "Input Power Select"
- note removed: "Jumper:"
- note removed: "Medium current MOSFET outputs (24V/6A)"
- note removed: "SPI Expansion"
- note removed: "Serial Expansion"
- note removed: "TO HBP"
- note removed: "TO HOTEND HEATER"
- note removed: "TO PRINT FAN"
- note removed: "Thermistor Inputs"
- moved on the sheet: C11, C14, C15, C6, C7, C8, C9, D2, D3, M1, M2, M3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

Commit message: Final rev C design files
Parts:
- removed P15, P16: CONN_02X02, Pin_Headers:Pin_Header_Straight_2x02, symbol CONN_02X02
- added C16: .1UF, Capacitors_SMD:C_0805_HandSoldering, symbol C
- added P12, P18: JST-PH, RAMPZ:JST_PH_2POS, symbol CONN_01X02
- added P15, P16: DUPONT, Pin_Headers:Pin_Header_Straight_1x02, symbol CONN_01X02
- added P26: CONN_02X04, RAMPZ:PINHEADER_2X4_SMD, symbol CONN_02X04
- added U3: TLV70033DDC, SOT-23-5, symbol TLV70033DDC
- C12: value .1 -> .1UF; footprint Capacitors_SMD:C_1206_HandSoldering -> Capacitors_SMD:C_0805_HandSoldering
- D11, D7, D8: PN (none) -> D-340
- Q2, Q4, Q6: value IRLM6346 -> IRLML6346
- R1, R2, R3, R7: value 4.7k -> 4.7K; footprint Resistors_SMD:R_0805 -> Resistors_SMD:R_0805_HandSoldering
- R10: value 4.7K -> 2K
- R13, R14, R16: value 4.7k -> 4.7K
- R4: footprint Resistors_SMD:R_0805 -> Resistors_SMD:R_0805_HandSoldering
- R5, R6: value 10K -> 4.7K; footprint (none) -> Resistors_SMD:R_0805_HandSoldering
- RP1: value YC164-JR-0722RL -> YC164-JR-0733RL
- RP2: value YC164-JR-07100KL -> YC164-JR-07150KL
Connections:
- net +12V: now also P12.2 (P2), P15.2 (P2), P16.2 (P2), P18.2 (P2)
- net BED_EN: now also R11.1
- net FAN_EN: now also RP2.2 (P2), SHIELD1.9; no longer RP2.3 (P3), SHIELD1.11
- net FE1_D: now also P12.1 (P1), P15.1 (P1)
- net FE2_D: now also P16.1 (P1), P18.1 (P1)
- net GND: now also C16.2, P26.2 (P2), U3.2 (GND)
- net HOTEND_EN: now also SHIELD1.10; no longer SHIELD1.9
- net RX1: now also P26.1 (P1)
- net VCC: now also U3.1 (IN), U3.3 (EN)
- net HOTEND2_EN: now reaches SHIELD1.2
- net HOTEND2_EN: now also RP1.3 (P3), RP2.4 (P4)
- net FAN2_EN: now reaches SHIELD1.7
- net FAN2_EN: now also RP1.1 (P1), RP2.3 (P3)
- net at Q3.1 (G), R9.1: no longer R11.1
- net TX1_S: now reaches R15.1, R16.1, SER1.4 (P4)
- net TX1_S: now also P26.8 (P8)
- removed net FET3_EN: RP1.3 (P3), RP2.2 (P2), SHIELD1.10
- removed net FET5_EN: RP1.1 (P1), RP2.4 (P4), SHIELD1.12
- new net: C16.1, P26.3 (P3), P26.7 (P7), U3.5 (OUT)
Other:
- note added: "150K"
- note added: "C"
- note added: "Design by Marty Rice <mrice411@gmail.com>\nThis work is licensed under a Creative Commons Attribution-ShareAlike \n4.0 International License."
- note added: "ESP8266 experimental socket"
- note added: "KEYSTONE 3519"
- note added: "Pololu Stepper Motor Sockets"
- note added: "Remove R14 and R16\nif interfacing to 5V serial\ndevice(s)."
- note removed: "100K"
- note removed: "EEE-1JA470UP"
- note removed: "Stepper Motor Sockets"
- moved on the sheet: R11, R15, R9, SER1

Commit message: update rev e files
Parts:
- removed D7: SS36, Diodes_SMD:SMA_Handsoldering, symbol D_Schottky
- removed P15: DUPONT, Pin_Headers:Pin_Header_Straight_1x02, symbol CONN_01X02
- removed RL1: SSR_2, RAMPZ:I4-PAC, symbol SSR_2
- removed RP1: YC164-JR-0733RL, RAMPZ:RESARY_4_CTS_744, symbol R_PACK4
- removed RP3: YC164-JR-073K3L, RAMPZ:RESARY_4_CTS_744, symbol R_PACK4
- added C17: 10nF, Capacitors_SMD:C_1206_HandSoldering, symbol C
- added D1: SBRT20M60SP5-7, RAMPZ:POWERDI5, symbol schottky3
- added F1, F2, F3: 0ZCJ0020FF2E, Fuse_Holders_and_Fuses:Fuse_SMD1206_Wave, symbol FUSE
- added R17, R18: 360, Resistors_SMD:R_0805_HandSoldering, symbol R
- added R19, R31, R32: 50, Resistors_SMD:R_0805_HandSoldering, symbol R
- added R27, R28, R29, R30: 4.7K, Resistors_SMD:R_0805_HandSoldering, symbol R
- added U4: MOC3061M, RAMPZ:6SMD, symbol MOC3061M
- added U5: TRIAC, TO_SOT_Packages_SMD:TO-252-2Lead, symbol TRIAC
- C13: value 15nF -> 10nF; footprint Capacitors_SMD:C_0805_HandSoldering -> Capacitors_SMD:C_1206_HandSoldering
- D11: value SS36 -> MBR0560; footprint Diodes_SMD:SMA_Handsoldering -> Diodes_SMD:SOD-123; PN D-340 -> (none)
- EXP1, EXP2: footprint Connect:IDC_Header_Straight_10pins -> RAMPZ:IDC_Header_Straight_10pins_DUAL
- P12: value JST-PH -> JST-XH; footprint RAMPZ:JST_PH_2POS -> RAMPZ:JST_XH_2POS
- R10: value 2K -> 200
- R9: value 10 -> 50
Connections:
- net FE1_G is gone; now on net FAN_EN: Q2.1 (G)
- net FE2_G is gone; now on net FAN2_EN: Q6.1 (G)
- net +12V: now also F3.2, R27.2, R28.2; no longer P5.6 (P6), P5.8 (P8), P6.2 (P2), P8.2 (P2)
- net +VPSU: now also D1.3, R29.2, R30.2
- net AM_VIN: now also F1.1; no longer R4.1, SHIELD1.V_IN
- net GND: now also D1.1, D1.2
- net HE1_G: now also R32.1
- net HE2_G: now also R31.1
- net HOTEND2_EN: now also R31.2
- net HOTEND_EN: now also R32.2
- net VCC: now also F2.2; no longer DRV_E0.2 (VDD), DRV_E1.2 (VDD), DRV_X1.2 (VDD), DRV_Y1.2 (VDD), DRV_Z1.2 (VDD), J1.1 (P1), J1.3 (P3), J1.5 (P5), J2.1 (P1), J2.3 (P3), J2.5 (P5), J3.1 (P1), J3.3 (P3), J3.5 (P5), J4.1 (P1), J4.3 (P3), J4.5 (P5), J5.1 (P1), J5.3 (P3), J5.5 (P5), R1.1, R2.1, R20.1, R21.1, R22.1, R23.1, R24.1, R3.1, R7.1
- net +5VL: now reaches SHIELD1.5V
- net +5VL: now also R1.1, R2.1, R3.1, R7.1
- net at D5.2 (A): now also R28.1
- net at D6.2 (A): now also R30.1
- net at D9.2 (A): now also R29.1
- net at D10.2 (A): now also R27.1
- net at D3.1 (K): now also U4.1
- net at Q4.3 (D): now also U4.2
- net at P14.1 (P1), P14.2 (P2): now also R17.2, R19.2, U5.1
- net at P13.1 (P1), P13.2 (P2): now also C17.1, R18.1, U5.2
- new net: F1.2, R4.1, SHIELD1.V_IN
- new net: F3.1, P5.6 (P6), P5.8 (P8), P6.2 (P2), P8.2 (P2)
- new net: R17.1, U4.4, U5.3
- new net: R18.2, U4.6
- new net: C17.2, R19.1
- new net DRV_VCC: DRV_E0.2 (VDD), DRV_E1.2 (VDD), DRV_X1.2 (VDD), DRV_Y1.2 (VDD), DRV_Z1.2 (VDD), F2.1, J1.1 (P1), J1.3 (P3), J1.5 (P5), J2.1 (P1), J2.3 (P3), J2.5 (P5), J3.1 (P1), J3.3 (P3), J3.5 (P5), J4.1 (P1), J4.3 (P3), J4.5 (P5), J5.1 (P1), J5.3 (P3), J5.5 (P5), R20.1, R21.1, R22.1, R23.1, R24.1
Other:
- note added: "HOT"
- note added: "LOAD"
- note added: "POWER ON"
- note added: "TRIAC FOR AC LOADS"
- note removed: "POWER"
- note removed: "SSR FOR AC LOADS"
- moved on the sheet: D10, D2, D3, D6, D9, P13, P14, P7, Q4, R10, R4, R5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
